Commit message: minor fixes and fixed URDFs

File: urdf/five_point_planar_robot.urdf (robot description, URDF)
Before this commit: robot point_planar_robot, 3 links, 2 joints
Links:
- added link link4
- added link link5
- added link link6
- added link link7
- added link link8
Joints:
- added joint joint3: type revolute, parent link3, child link4, origin xyz=0 0 0 rpy=0 0 0, axis 0 0 1
- added joint joint4: type revolute, parent link4, child link5, origin xyz=0 5 0 rpy=0 0 0, axis 0 0 1
- added joint joint5: type revolute, parent link5, child link6, origin xyz=5 0 0 rpy=0 0 0, axis 0 0 1
- added joint joint6: type revolute, parent link6, child link7, origin xyz=0 5 0 rpy=0 0 0, axis 0 0 1
- added joint joint7: type fixed, parent link7, child link8, origin xyz=5 0 0 rpy=0 0 0, axis 0 0 1
